File: PCB/ControlCabinet/ControlCabinet.kicad_pcb (KiCad board)
At the start: 4 copper layers, 153.7 x 115.6 mm, 63 parts, among them J1 Screw_Terminal_01x03, J10 Conn_01x08, J11 Conn_01x08, J12 Conn_01x08, J13 Conn_01x08, J14 Conn_01x08, J15 Conn_01x08, J16 Conn_01x04, J17 Conn_01x02, J18 Conn_01x04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

Commit message: Progress report Brezen + zavisle soubory
Other:
- board text added: "Vref = Current Limit/2"
